File: hardware/kicad/12_aux_rails.kicad_sch (KiCad schematic)
At the start: 20 parts, among them U1201 LM5164 (candidate), U1202 TLV75533

Commit message: sem-motor-controller v0.3: vehicle-interface provenance, transport-neutral core, clock trees, schematic checks
Provenance: the Cornell repositories are reference projects. Every place
that treated CHUDS / CAN FD / its VCU / 40 MHz as our vehicle is relabelled
or corrected (docs/PROVENANCE_AUDIT.md); the v0.2 checkpoint is preserved
with an errata banner.

Firmware: the core is transport-neutral (mc_core_on_msg_rx /
mc_core_msg_tx_poll / mc_core_on_link_state). CAN is one binding
(src/transport/mc_can_binding.c) whose 64-identifier block base is the new
calibration parameter supervision.can_id_base (id 164, rule 40, null in the
unconfigured config). ADR-0012. Tests: block relocation with a full ECO
engagement at 0x500, neutral API, rule-40 C/Python parity.

Clocking: tools/clock_tree.py evaluates 28 complete clock trees x 4 bus
cases from ST register widths and HAL ranges; the v0.2 "40 MHz required"
claim is withdrawn and the crystal is unselected until the bus is known.

Schematic: INA228 pins renumbered (KiCad-library cross-check, secondary);
DRV8353S stays an explicit placeholder; crystal unselected; PWR_FLAGs added
after a new pin-type check (not an ERC) found 6 undriven-rail errors.
Real KiCad ERC not run (KiCad 7 has no CLI ERC; tools/run_kicad_erc.sh).

Telematics: combined architecture with the STM32U575 / CAN 2.0B / LTE-MQTT
proposal (supervisor and CSIA placement, torque-request and driver-
authorization paths, pit/cloud outside the control chain), interface
difference table, generated DBC, logging-capacity and auxiliary-power
budget. Validation language separates command ceilings, envelope ramp,
phase current and battery current. CSIA: component attribution and a
next-evaluation plan; frozen results unchanged, nothing re-run.

Verified on the host: ctest 6/6 (4,006 checks), pytest 199 passed,
ARM core build 0 warnings, generators current, KiCad connectivity 0
problems. Nothing on hardware.

Co-Authored-By: Claude Opus 5.5 <noreply@anthropic.com>
Claude-Ses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
Changed lines of the file:
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@@
     (effects (font (size 1.27 1.27)) (justify right))
   )
-  (symbol (lib_id "Regulator_Switching:LM5164DDA") (at 83.82000000000001 68.58 0) (unit 1)
-    (in_bom yes) (on_board yes)
-    (property "Reference" "U1201" (id 0) (at 83.82000000000001 63.5 0)
-      (effects (font (size 1.27 1.27)))
-    )
-    (property "Value" "LM5164 (candidate)" (id 1) (at 83.82000000000001 73.66 0)
-      (effects (font (size 1.27 1.27)))
-    )
-    (property "Footprint" "" (id 2) (at 83.82000000000001 68.58 0)
-      (effects (font (size 1.27 1.27)) hide)
-    )
-    (property "Datasheet" "" (id 3) (at 83.82000000000001 68.58 0)
-      (effects (font (size 1.27 1.27)) hide)
-    )
-    (property "Status" "CANDIDATE (100 V input class - verify)" (id 4) (at 83.82000000000001 68.58 0)
-      (effects (font (size 1.27 1.27)) hide)
-    )
-    (property "MPN" "LM5164DDAR" (id 5) (at 83.82000000000001 68.58 0)
+  (symbol (lib_id "Regulator_Switching:LM5164DDA") (at 83.82 68.58 0) (unit 1)
+    (in_bom yes) (on_board yes)
+    (property "Reference" "U1201" (id 0) (at 83.82 63.5 0)
+      (effects (font (size 1.27 1.27)))
+    )
+    (property "Value" "LM5164 (candidate)" (id 1) (at 83.82 73.66 0)
+      (effects (font (size 1.27 1.27)))
+    )
+    (property "Footprint" "" (id 2) (at 83.82 68.58 0)
+      (effects (font (size 1.27 1.27)) hide)
+    )
+    (property "Datasheet" "" (id 3) (at 83.82 68.58 0)
+      (effects (font (size 1.27 1.27)) hide)
+    )
+    (property "Status" "CANDIDATE (100 V input class - verify)" (id 4) (at 83.82 68.58 0)
+      (effects (font (size 1.27 1.27)) hide)
+    )
+    (property "MPN" "LM5164DDAR" (id 5) (at 83.82 68.58 0)
       (effects (font (size 1.27 1.27)) hide)
     )
@@
     (pin "2")
   )
-  (symbol (lib_id "Device:R") (at 335.28000000000003 66.04 0) (unit 1)
-    (in_bom yes) (on_board yes)
-    (property "Reference" "R1202" (id 0) (at 335.28000000000003 60.96000000000001 0)
-      (effects (font (size 1.27 1.27)))
-    )
-    (property "Value" "UNRESOLVED UVLO bottom" (id 1) (at 335.28000000000003 71.12 0)
-      (effects (font (size 1.27 1.27)))
-    )
-    (property "Footprint" "" (id 2) (at 335.28000000000003 66.04 0)
-      (effects (font (size 1.27 1.27)) hide)
-    )
-    (property "Datasheet" "" (id 3) (at 335.28000000000003 66.04 0)
-      (effects (font (size 1.27 1.27)) hide)
-    )
-    (property "Status" "UNRESOLVED" (id 4) (at 335.28000000000003 66.04 0)
+  (symbol (lib_id "Device:R") (at 335.28 66.04 0) (unit 1)
+    (in_bom yes) (on_board yes)
+    (property "Reference" "R1202" (id 0) (at 335.28 60.96000000000001 0)
+      (effects (font (size 1.27 1.27)))
+    )
+    (property "Value" "UNRESOLVED UVLO bottom" (id 1) (at 335.28 71.12 0)
+      (effects (font (size 1.27 1.27)))
+    )
+    (property "Footprint" "" (id 2) (at 335.28 66.04 0)
+      (effects (font (size 1.27 1.27)) hide)
+    )
+    (property "Datasheet" "" (id 3) (at 335.28 66.04 0)
+      (effects (font (size 1.27 1.27)) hide)
+    )
+    (property "Status" "UNRESOLVED" (id 4) (at 335.28 66.04 0)
       (effects (font (size 1.27 1.27)) hide)
     )
@@
     (pin "2")
   )
-  (symbol (lib_id "Device:C") (at 248.92000000000002 111.76 0) (unit 1)
-    (in_bom yes) (on_board yes)
-    (property "Reference" "C1204" (id 0) (at 248.92000000000002 106.68 0)
-      (effects (font (size 1.27 1.27)))
-    )
-    (property "Value" "22uF" (id 1) (at 248.92000000000002 116.84 0)
-      (effects (font (size 1.27 1.27)))
-    )
-    (property "Footprint" "" (id 2) (at 248.92000000000002 111.76 0)
-      (effects (font (size 1.27 1.27)) hide)
-    )
-    (property "Datasheet" "" (id 3) (at 248.92000000000002 111.76 0)
-      (effects (font (size 1.27 1.27)) hide)
-    )
-    (property "Status" "design value" (id 4) (at 248.92000000000002 111.76 0)
+  (symbol (lib_id "Device:C") (at 248.92 111.76 0) (unit 1)
+    (in_bom yes) (on_board yes)
+    (property "Reference" "C1204" (id 0) (at 248.92 106.68 0)
+      (effects (font (size 1.27 1.27)))
+    )
+    (property "Value" "22uF" (id 1) (at 248.92 116.84 0)
+      (effects (font (size 1.27 1.27)))
+    )
+    (property "Footprint" "" (id 2) (at 248.92 111.76 0)
+      (effects (font (size 1.27 1.27)) hide)
+    )
+    (property "Datasheet" "" (id 3) (at 248.92 111.76 0)
+      (effects (font (size 1.27 1.27)) hide)
+    )
+    (property "Status" "design value" (id 4) (at 248.92 111.76 0)
       (effects (font (size 1.27 1.27)) hide)
     )
@@
     (pin "2")
   )
-  (symbol (lib_id "Device:R") (at 370.84000000000003 111.76 0) (unit 1)
-    (in_bom yes) (on_board yes)
-    (property "Reference" "R1206" (id 0) (at 370.84000000000003 106.68 0)
-      (effects (font (size 1.27 1.27)))
-    )
-    (property "Value" "100k" (id 1) (at 370.84000000000003 116.84 0)
-      (effects (font (size 1.27 1.27)))
-    )
-    (property "Footprint" "" (id 2) (at 370.84000000000003 111.76 0)
-      (effects (font (size 1.27 1.27)) hide)
-    )
-    (property "Datasheet" "" (id 3) (at 370.84000000000003 111.76 0)
-      (effects (font (size 1.27 1.27)) hide)
-    )
-    (property "Status" "design value" (id 4) (at 370.84000000000003 111.76 0)
-      (effects (font (size 1.27 1.27)) hide)
-    )
+  (symbol (lib_id "Device:R") (at 370.84 111.76 0) (unit 1)
+    (in_bom yes) (on_board yes)
+    (property "Reference" "R1206" (id 0) (at 370.84 106.68 0)
+      (effects (font (size 1.27 1.27)))
+    )
+    (property "Value" "100k" (id 1) (at 370.84 116.84 0)
+      (effects (font (size 1.27 1.27)))
+    )
+    (property "Footprint" "" (id 2) (at 370.84 111.76 0)
+      (effects (font (size 1.27 1.27)) hide)
+    )
+    (property "Datasheet" "" (id 3) (at 370.84 111.76 0)
+      (effects (font (size 1.27 1.27)) hide)
+    )
+    (property "Status" "design value" (id 4) (at 370.84 111.76 0)
+      (effects (font (size 1.27 1.27)) hide)
+    )
