File: hardware/kicad/01_power_input.kicad_sch (KiCad schematic)
At the start: 13 parts, among them J101 BATTERY_IN, Q101 UNRESOLVED bypass P-FET, Q102 UNRESOLVED small-signal N-FET, U101 UNRESOLVED reverse-polarity p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

Commit message: sem-motor-controller v0.3: vehicle-interface provenance, transport-neutral core, clock trees, schematic checks
Provenance: the Cornell repositories are reference projects. Every place
that treated CHUDS / CAN FD / its VCU / 40 MHz as our vehicle is relabelled
or corrected (docs/PROVENANCE_AUDIT.md); the v0.2 checkpoint is preserved
with an errata banner.

Firmware: the core is transport-neutral (mc_core_on_msg_rx /
mc_core_msg_tx_poll / mc_core_on_link_state). CAN is one binding
(src/transport/mc_can_binding.c) whose 64-identifier block base is the new
calibration parameter supervision.can_id_base (id 164, rule 40, null in the
unconfigured config). ADR-0012. Tests: block relocation with a full ECO
engagement at 0x500, neutral API, rule-40 C/Python parity.

Clocking: tools/clock_tree.py evaluates 28 complete clock trees x 4 bus
cases from ST register widths and HAL ranges; the v0.2 "40 MHz required"
claim is withdrawn and the crystal is unselected until the bus is known.

Schematic: INA228 pins renumbered (KiCad-library cross-check, secondary);
DRV8353S stays an explicit placeholder; crystal unselected; PWR_FLAGs added
after a new pin-type check (not an ERC) found 6 undriven-rail errors.
Real KiCad ERC not run (KiCad 7 has no CLI ERC; tools/run_kicad_erc.sh).

Telematics: combined architecture with the STM32U575 / CAN 2.0B / LTE-MQTT
proposal (supervisor and CSIA placement, torque-request and driver-
authorization paths, pit/cloud outside the control chain), interface
difference table, generated DBC, logging-capacity and auxiliary-power
budget. Validation language separates command ceilings, envelope ramp,
phase current and battery current. CSIA: component attribution and a
next-evaluation plan; frozen results unchanged, nothing re-run.

Verified on the host: ctest 6/6 (4,006 checks), pytest 199 passed,
ARM core build 0 warnings, generators current, KiCad connectivity 0
problems. Nothing on hardware.

Co-Authored-By: Claude Opus 5.5 <noreply@anthropic.com>
Claude-Ses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
Changed lines of the file:
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@@
+    (effects (font (size 1.27 1.27)) (justify right))
+  )
+  (global_label "VBAT_PROT" (shape passive) (at 452.12 96.52 270)
+    (effects (font (size 1.27 1.27)) (justify right))
+  )
+  (global_label "VDC" (shape passive) (at 71.12 132.08 270)
+    (effects (font (size 1.27 1.27)) (justify right))
+  )
+  (global_label "PGND" (shape passive) (at 129.54 132.08 270)
+    (effects (font (size 1.27 1.27)) (justify right))
+  )
+  (global_label "GND" (shape passive) (at 190.5 132.08 270)
+    (effects (font (size 1.27 1.27)) (justify right))
+  )
+  (global_label "+5V" (shape passive) (at 248.92 132.08 270)
+    (effects (font (size 1.27 1.27)) (justify right))
+  )
+  (global_label "+3V3A" (shape passive) (at 309.88 132.08 270)
     (effects (font (size 1.27 1.27)) (justify right))
   )
@@
     (pin "2")
   )
-  (symbol (lib_id "Device:R_Shunt") (at 398.78000000000003 66.04 0) (unit 1)
-    (in_bom yes) (on_board yes)
-    (property "Reference" "R101" (id 0) (at 398.78000000000003 60.96000000000001 0)
-      (effects (font (size 1.27 1.27)))
-    )
-    (property "Value" "UNRESOLVED bus shunt" (id 1) (at 398.78000000000003 71.12 0)
-      (effects (font (size 1.27 1.27)))
-    )
-    (property "Footprint" "" (id 2) (at 398.78000000000003 66.04 0)
-      (effects (font (size 1.27 1.27)) hide)
-    )
-    (property "Datasheet" "" (id 3) (at 398.78000000000003 66.04 0)
-      (effects (font (size 1.27 1.27)) hide)
-    )
-    (property "Status" "UNRESOLVED" (id 4) (at 398.78000000000003 66.04 0)
-      (effects (font (size 1.27 1.27)) hide)
-    )
-    (property "Rating_basis" "I_batt,max into INA228 full-scale range; Kelvin sense pads" (id 5) (at 398.78000000000003 66.04 0)
+  (symbol (lib_id "Device:R_Shunt") (at 398.78 66.04 0) (unit 1)
+    (in_bom yes) (on_board yes)
+    (property "Reference" "R101" (id 0) (at 398.78 60.96000000000001 0)
+      (effects (font (size 1.27 1.27)))
+    )
+    (property "Value" "UNRESOLVED bus shunt" (id 1) (at 398.78 71.12 0)
+      (effects (font (size 1.27 1.27)))
+    )
+    (property "Footprint" "" (id 2) (at 398.78 66.04 0)
+      (effects (font (size 1.27 1.27)) hide)
+    )
+    (property "Datasheet" "" (id 3) (at 398.78 66.04 0)
+      (effects (font (size 1.27 1.27)) hide)
+    )
+    (property "Status" "UNRESOLVED" (id 4) (at 398.78 66.04 0)
+      (effects (font (size 1.27 1.27)) hide)
+    )
+    (property "Rating_basis" "I_batt,max into INA228 full-scale range; Kelvin sense pads" (id 5) (at 398.78 66.04 0)
       (effects (font (size 1.27 1.27)) hide)
     )
@@
     (pin "4")
   )
-  (symbol (lib_id "Device:R") (at 462.28000000000003 66.04 0) (unit 1)
-    (in_bom yes) (on_board yes)
-    (property "Reference" "R102" (id 0) (at 462.28000000000003 60.96000000000001 0)
-      (effects (font (size 1.27 1.27)))
-    )
-    (property "Value" "UNRESOLVED precharge R" (id 1) (at 462.28000000000003 71.12 0)
-      (effects (font (size 1.27 1.27)))
-    )
-    (property "Footprint" "" (id 2) (at 462.28000000000003 66.04 0)
-      (effects (font (size 1.27 1.27)) hide)
-    )
-    (property "Datasheet" "" (id 3) (at 462.28000000000003 66.04 0)
-      (effects (font (size 1.27 1.27)) hide)
-    )
-    (property "Status" "UNRESOLVED" (id 4) (at 462.28000000000003 66.04 0)
-      (effects (font (size 1.27 1.27)) hide)
-    )
-    (property "Rating_basis" "C_link, V_bat,max, precharge time; pulse energy 0.5*C*V^2 per attempt" (id 5) (at 462.28000000000003 66.04 0)
+  (symbol (lib_id "Device:R") (at 462.28 66.04 0) (unit 1)
+    (in_bom yes) (on_board yes)
+    (property "Reference" "R102" (id 0) (at 462.28 60.96000000000001 0)
+      (effects (font (size 1.27 1.27)))
+    )
+    (property "Value" "UNRESOLVED precharge R" (id 1) (at 462.28 71.12 0)
+      (effects (font (size 1.27 1.27)))
+    )
+    (property "Footprint" "" (id 2) (at 462.28 66.04 0)
+      (effects (font (size 1.27 1.27)) hide)
+    )
+    (property "Datasheet" "" (id 3) (at 462.28 66.04 0)
+      (effects (font (size 1.27 1.27)) hide)
+    )
+    (property "Status" "UNRESOLVED" (id 4) (at 462.28 66.04 0)
+      (effects (font (size 1.27 1.27)) hide)
+    )
+    (property "Rating_basis" "C_link, V_bat,max, precharge time; pulse energy 0.5*C*V^2 per attempt" (id 5) (at 462.28 66.04 0)
       (effects (font (size 1.27 1.27)) hide)
     )
@@
     (pin "2")
   )
+  (symbol (lib_id "power:PWR_FLAG") (at 452.12 96.52 0) (unit 1)
+    (in_bom yes) (on_board yes)
+    (property "Reference" "#FLG101" (id 0) (at 452.12 91.44 0)
+      (effects (font (size 1.27 1.27)))
+    )
+    (property "Value" "PWR_FLAG" (id 1) (at 452.12 101.6 0)
+      (effects (font (size 1.27 1.27)))
+    )
+    (property "Footprint" "" (id 2) (at 452.12 96.52 0)
+      (effects (font (size 1.27 1.27)) hide)
+    )
+    (property "Datasheet" "" (id 3) (at 452.12 96.52 0)
+      (effects (font (size 1.27 1.27)) hide)
+    )
+    (property "Status" "ERC marker" (id 4) (at 452.12 96.52 0)
+      (effects (font (size 1.27 1.27)) hide)
+    )
+    (pin "1")
+  )
+  (symbol (lib_id "power:PWR_FLAG") (at 71.12 132.08 0) (unit 1)
+    (in_bom yes) (on_board yes)
+    (property "Reference" "#FLG102" (id 0) (at 71.12 127.00000000000001 0)
+      (effects (font (size 1.27 1.27)))
+    )
+    (property "Value" "PWR_FLAG" (id 1) (at 71.12 137.16000000000003 0)
+      (effects (font (size 1.27 1.27)))
+    )
+    (property "Footprint" "" (id 2) (at 71.12 132.08 0)
+      (effects (font (size 1.27 1.27)) hide)
+    )
+    (property "Datasheet" "" (id 3) (at 71.12 132.08 0)
+      (effects (font (size 1.27 1.27)) hide)
+    )
+    (property "Status" "ERC marker" (id 4) (at 71.12 132.08 0)
+      (effects (font (size 1.27 1.27)) hide)
+    )
+    (pin "1")
+  )
+  (symbol (lib_id "power:PWR_FLAG") (at 129.54 132.08 0) (unit 1)
+    (in_bom yes) (on_board yes)
+    (property "Reference" "#FLG103" (id 0) (at 129.54 127.00000000000001 0)
+      (effects (font (size 1.27 1.27)))
+    )
+    (property "Value" "PWR_FLAG" (id 1) (at 129.54 137.16000000000003 0)
+      (effects (font (size 1.27 1.27)))
+    )
+    (property "Footprint" "" (id 2) (at 129.54 132.08 0)
+      (effects (font (size 1.27 1.27)) hide)
+    )
+    (property "Datasheet" "" (id 3) (at 129.54 132.08 0)
+      (effects (font (size 1.27 1.27)) hide)
+    )
+    (property "Status" "ERC marker" (id 4) (at 129.54 132.08 0)
+      (effects (font (size 1.27 1.27)) hide)
+    )
+    (pin "1")
+  )
+  (symbol (lib_id "power:PWR_FLAG") (at 190.5 132.08 0) (unit 1)
+    (in_bom yes) (on_board yes)
+    (property "Reference" "#FLG104" (id 0) (at 190.5 127.00000000000001 0)
+      (effects (font (size 1.27 1.27)))
+    )
+    (property "Value" "PWR_FLAG" (id 1) (at 190.5 137.16000000000003 0)
+      (effects (font (size 1.27 1.27)))
+    )
+    (property "Footprint" "" (id 2) (at 190.5 132.08 0)
+      (effects (font (size 1.27 1.27)) hide)
+    )
+    (property "Datasheet" "" (id 3) (at 190.5 132.08 0)
+      (effects (font (size 1.27 1.27)) hide)
+    )
+    (property "Status" "ERC marker" (id 4) (at 190.5 132.08 0)
+      (effects (font (size 1.27 1.27)) hide)
+    )
+    (pin "1")
+  )
+  (symbol (lib_id "power:PWR_FLAG") (at 248.92 132.08 0) (unit 1)
+    (in_bom yes) (on_board yes)
+    (property "Reference" "#FLG105" (id 0) (at 248.92 127.00000000000001 0)
+      (effects (font (size 1.27 1.27)))
+    )
+    (property "Value" "PWR_FLAG" (id 1) (at 248.92 137.16000000000003 0)
+      (effects (font (size 1.27 1.27)))
+    )
+    (property "Footprint" "" (id 2) (at 248.92 132.08 0)
+      (effects (font (size 1.27 1.27)) hide)
+    )
+    (property "Datasheet" "" (id 3) (at 248.92 132.08 0)
+      (effects (font (size 1.27 1.27)) hide)
+    )
+    (property "Status" "ERC marker" (id 4) (at 248.92 132.08 0)
+      (effects (font (size 1.27 1.27)) hide)
+    )
+    (pin "1")
+  )
+  (symbol (lib_id "power:PWR_FLAG") (at 309.88 132.08 0) (unit 1)
+    (in_bom yes) (on_board yes)
+    (property "Reference" "#FLG106" (id 0) (at 309.88 127.00000000000001 0)
+      (effects (font (size 1.27 1.27)))
+    )
+    (property "Value" "PWR_FLAG" (id 1) (at 309.88 137.16000000000003 0)
+      (effects (font (size 1.27 1.27)))
+    )
+    (property "Footprint" "" (id 2) (at 309.88 132.08 0)
+      (effects (font (size 1.27 1.27)) hide)
+    )
+    (property "Datasheet" "" (id 3) (at 309.88 132.08 0)
+      (effects (font (size 1.27 1.27)) hide)
+    )
+    (property "Status" "ERC marker" (id 4) (at 309.88 132.08 0)
+      (effects (font (size 1.27 1.27)) hide)
+    )
+    (pin "1")
+  )
   (sheet_instances

Commit message: hardware: design review, OV comparator hysteresis fix, test points, KiCad 8.0.9 libraries
hardware/review/DESIGN_REVIEW.md reviews the draft item by item (gate
driver, MOSFETs, DC link, current sensing, hardware overcurrent,
over/undervoltage, temperature, precharge, enable defaults and
watchdog, emergency interface, DC-DC, CAN, clock, debug and test
points) with an evidence level per statement, and records what each
open item needs.

Schematic changes that need no vehicle data:
- the over-voltage comparator's hysteresis resistor went straight onto
  the TL431 node, whose low impedance made the hysteresis undefined;
  the + input is now fed through 10 k and 390 k from the output sets
  -2.5 % / +0.8 % around the reference;
- the TL431 bias is 470 ohm (1.7 mA) instead of 1 k (0.8 mA), above
  its minimum cathode current (recalled; to confirm in the datasheet);
- the six pull-downs on the gate-signal inputs are fitted until the
  driver's own pull-downs are verified;
- 21 test points for the signals the acceptance procedures probe.
Connectivity: 136 intended nets, 0 problems; pin types 0 findings;
consistency 14 PASS, 4 OPEN.

The nine KiCad 8.0.9 ERC warnings were each compared with the library:
PWR_FLAG pin name, TL431 drawing, STM32G474 symbol geometry and the
NUP2105L datasheet URL changed between the 7.0.11 library the
schematic embedded and 8.0.9; no pin number, connected name, type or
net changed. The schematic is now generated from a pinned, SHA-256
checked copy of the 8.0.9 libraries (tools/fetch_kicad_symbols.py),
which the ERC also reads; KiCad 8's (hide yes) spelling is converted
for kiutils so no field becomes visible. Both CI jobs use KiCad 8.

Firmware: the brake switch type is a calibration value; a separate
bench image (semmc_stm32g474_pwmtest) switches the gate signals at
fixed duties with DRV_ENABLE held low for acceptance stage 4; g_bench
also reports the input states.

Co-Authored-By: Claude Opus 5.5 <noreply@anthropic.com>
Claude-Session: https:/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
Parts:
- added TP101: PRECHG_EN, symbol Connector:TestPoint
Connections:
- net PRECHG_EN: now also TP101.1
Changed lines of the file:
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@@
     (effects (font (size 1.27 1.27)) (justify right))
   )
-  (global_label "VBAT_PROT" (shape passive) (at 452.12 96.52 270)
-    (effects (font (size 1.27 1.27)) (justify right))
-  )
-  (global_label "VDC" (shape passive) (at 71.12 132.08 270)
-    (effects (font (size 1.27 1.27)) (justify right))
-  )
-  (global_label "PGND" (shape passive) (at 129.54 132.08 270)
-    (effects (font (size 1.27 1.27)) (justify right))
-  )
-  (global_label "GND" (shape passive) (at 190.5 132.08 270)
-    (effects (font (size 1.27 1.27)) (justify right))
-  )
-  (global_label "+5V" (shape passive) (at 248.92 132.08 270)
-    (effects (font (size 1.27 1.27)) (justify right))
-  )
-  (global_label "+3V3A" (shape passive) (at 309.88 132.08 270)
+  (global_label "VBAT_PROT" (shape passive) (at 71.12 132.08 270)
+    (effects (font (size 1.27 1.27)) (justify right))
+  )
+  (global_label "VDC" (shape passive) (at 129.54 132.08 270)
+    (effects (font (size 1.27 1.27)) (justify right))
+  )
+  (global_label "PGND" (shape passive) (at 190.5 132.08 270)
+    (effects (font (size 1.27 1.27)) (justify right))
+  )
+  (global_label "GND" (shape passive) (at 248.92 132.08 270)
+    (effects (font (size 1.27 1.27)) (justify right))
+  )
+  (global_label "+5V" (shape passive) (at 309.88 132.08 270)
+    (effects (font (size 1.27 1.27)) (justify right))
+  )
+  (global_label "+3V3A" (shape passive) (at 370.84 132.08 270)
     (effects (font (size 1.27 1.27)) (justify right))
   )
@@
     (effects (font (size 1.27 1.27)) (justify left))
   )
+  (hierarchical_label "PRECHG_EN" (shape bidirectional) (at 452.12 96.52 270)
+    (effects (font (size 1.27 1.27)) (justify right))
+  )
   (symbol (lib_id "Connector_Generic:Conn_01x02") (at 76.2 60.96 0) (unit 1)
     (in_bom yes) (on_board yes)
@@
     (pin "2")
   )
-  (symbol (lib_id "power:PWR_FLAG") (at 452.12 96.52 0) (unit 1)
-    (in_bom yes) (on_board yes)
-    (property "Reference" "#FLG101" (id 0) (at 452.12 91.44 0)
-      (effects (font (size 1.27 1.27)))
-    )
-    (property "Value" "PWR_FLAG" (id 1) (at 452.12 101.6 0)
+  (symbol (lib_id "Connector:TestPoint") (at 452.12 96.52 0) (unit 1)
+    (in_bom yes) (on_board yes)
+    (property "Reference" "TP101" (id 0) (at 452.12 91.44 0)
+      (effects (font (size 1.27 1.27)))
+    )
+    (property "Value" "PRECHG_EN" (id 1) (at 452.12 101.6 0)
       (effects (font (size 1.27 1.27)))
     )
@@
       (effects (font (size 1.27 1.27)) hide)
     )
-    (property "Status" "ERC marker" (id 4) (at 452.12 96.52 0)
+    (property "Status" "bench test point" (id 4) (at 452.12 96.52 0)
       (effects (font (size 1.27 1.27)) hide)
     )
@@
   (symbol (lib_id "power:PWR_FLAG") (at 71.12 132.08 0) (unit 1)
     (in_bom yes) (on_board yes)
-    (property "Reference" "#FLG102" (id 0) (at 71.12 127.00000000000001 0)
+    (property "Reference" "#FLG101" (id 0) (at 71.12 127.00000000000001 0)
       (effects (font (size 1.27 1.27)))
     )
@@
   (symbol (lib_id "power:PWR_FLAG") (at 129.54 132.08 0) (unit 1)
     (in_bom yes) (on_board yes)
-    (property "Reference" "#FLG103" (id 0) (at 129.54 127.00000000000001 0)
+    (property "Reference" "#FLG102" (id 0) (at 129.54 127.00000000000001 0)
       (effects (font (size 1.27 1.27)))
     )
@@
   (symbol (lib_id "power:PWR_FLAG") (at 190.5 132.08 0) (unit 1)
     (in_bom yes) (on_board yes)
-    (property "Reference" "#FLG104" (id 0) (at 190.5 127.00000000000001 0)
+    (property "Reference" "#FLG103" (id 0) (at 190.5 127.00000000000001 0)
       (effects (font (size 1.27 1.27)))
     )
@@
   (symbol (lib_id "power:PWR_FLAG") (at 248.92 132.08 0) (unit 1)
     (in_bom yes) (on_board yes)
-    (property "Reference" "#FLG105" (id 0) (at 248.92 127.00000000000001 0)
+    (property "Reference" "#FLG104" (id 0) (at 248.92 127.00000000000001 0)
       (effects (font (size 1.27 1.27)))
     )
@@
   (symbol (lib_id "power:PWR_FLAG") (at 309.88 132.08 0) (unit 1)
     (in_bom yes) (on_board yes)
-    (property "Reference" "#FLG106" (id 0) (at 309.88 127.00000000000001 0)
+    (property "Reference" "#FLG105" (id 0) (at 309.88 127.00000000000001 0)
       (effects (font (size 1.27 1.27)))
     )
@@
       (effects (font (size 1.27 1.27)) hide)
     )
+    (pin "1")
+  )
+  (symbol (lib_id "power:PWR_FLAG") (at 370.84 132.08 0) (unit 1)
+    (in_bom yes) (on_board yes)
+    (property "Reference" "#FLG106" (id 0) (at 370.84 127.00000000000001 0)
+      (effects (font (size 1.27 1.27)))
+    )
+    (property "Value" "PWR_FLAG" (id 1) (at 370.84 137.16000000000003 0)
+      (effects (font (size 1.27 1.27)))
+    )
+    (property "Footprint" "" (id 2) (at 370.84 132.08 0)
+      (effects (font (size 1.27 1.27)) hide)
+    )
+    (property "Datasheet" "" (id 3) (at 370.84 132.08 0)
+      (effects (font (size 1.27 1.27)) hide)
+    )
+    (property "Status" "ERC marker" (id 4) (at 370.84 132.08 0)
+      (effects (font (size 1.27 1.27)) hide)
+    )

Commit message: hardware: footprint disposition for every BOM line, 82 assigned and checked
hardware/footprints/assignments.yaml gives each of the 122 BOM lines one
disposition. 68 lines are generic parts defined by value and package and
get a verified footprint (37 without the test points); 14 are specific
devices whose footprint is assigned from the KiCad 8.0.9 library but whose
manufacturer package drawing is unread (the LM5164 land pattern is drawn
from ST's L5973D HSOP-8 and the LQFP-100 from NXP's SOT407-1, so both must
be compared); 40 have none and say why: 28 rating-dependent, 4 waiting for a
data sheet value or pin voltage, 6 connectors, 2 placeholder pinouts.
Before this change no line had a footprint.

tools/check_footprints.py fetches the 25 footprint files used, pins them by
SHA-256, and checks per reference: numbered pads equal the symbol's pin
numbers, courtyard and fabrication outline present (copper-only jumpers and
net ties excepted), SMD or through-hole, package in the name for chip
parts, the symbol's footprint filters (as KiCad's ERC does), and pin 1 = K
on diode and LED symbols. Mutation tests cover a wrong pad count, a filter
miss, a package mismatch, a missing reference and a verified line without
a footprint. Small passives on battery-voltage nets (R104, R201, R202,
R1201) were kept rating-dependent rather than given an 0603.

The generator writes the footprints into the schematic and a footprint
column into the draft BOM; hw_consistency adds BM3 (netlist footprint
equals the BOM line's); price_bom takes footprint and package from the
assignment. Pricing rules fixed where lines matched the wrong rule: LEDs
were priced as buck inductors, crystal load capacitors as 100 V MLCCs, the
UART bench header as a harness connector, the reset switch and the Zener
under one generic rule; 22 uF and 4.7 uF now 1206 and 0805 for DC bias. One
board's parts move from $89-$239 to $88-$233. A project fp-lib-table and
the CI and ERC steps fetch the pinned footprints so the ERC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
Parts:
- D102: footprint (none) -> Diode_SMD:D_SOD-123
- R103, R105: footprint (none) -> Resistor_SMD:R_0603_1608Metric
- TP101: footprint (none) -> TestPoint:TestPoint_Pad_D1.5mm
Changed lines of the file:
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@@
       (effects (font (size 1.27 1.27)))
     )
-    (property "Footprint" "" (id 2) (at 137.16 101.6 0)
+    (property "Footprint" "Resistor_SMD:R_0603_1608Metric" (id 2) (at 137.16 101.6 0)
       (effects (font (size 1.27 1.27)) hide)
     )
@@
       (effects (font (size 1.27 1.27)))
     )
-    (property "Footprint" "" (id 2) (at 200.66 96.52 0)
+    (property "Footprint" "Diode_SMD:D_SOD-123" (id 2) (at 200.66 96.52 0)
       (effects (font (size 1.27 1.27)) hide)
     )
@@
       (effects (font (size 1.27 1.27)))
     )
-    (property "Footprint" "" (id 2) (at 393.7 101.6 0)
+    (property "Footprint" "Resistor_SMD:R_0603_1608Metric" (id 2) (at 393.7 101.6 0)
       (effects (font (size 1.27 1.27)) hide)
     )
@@
       (effects (font (size 1.27 1.27)))
     )
-    (property "Footprint" "" (id 2) (at 452.12 96.52 0)
+    (property "Footprint" "TestPoint:TestPoint_Pad_D1.5mm" (id 2) (at 452.12 96.52 0)
       (effects (font (size 1.27 1.27)) hide)
     )
