File: hardware/kicad/03_bridge.kicad_sch (KiCad schematic)
At the start: 16 parts, among them J301 MOTOR_PHASES, Q301 UNRESOLVED N-MOSFET HS-A, Q302 UNRESOLVED N-MOSFET LS-A, Q303 UNRESOLVED N-MOSFET HS-B, Q304 UNRESOLVED N-MOSFET LS-B, Q305 UNRESOLVED N-MOSFET HS-C, Q306 UNRESOLVED N-MOSFET LS-C

Commit message: sem-motor-controller v0.3: vehicle-interface provenance, transport-neutral core, clock trees, schematic checks
Provenance: the Cornell repositories are reference projects. Every place
that treated CHUDS / CAN FD / its VCU / 40 MHz as our vehicle is relabelled
or corrected (docs/PROVENANCE_AUDIT.md); the v0.2 checkpoint is preserved
with an errata banner.

Firmware: the core is transport-neutral (mc_core_on_msg_rx /
mc_core_msg_tx_poll / mc_core_on_link_state). CAN is one binding
(src/transport/mc_can_binding.c) whose 64-identifier block base is the new
calibration parameter supervision.can_id_base (id 164, rule 40, null in the
unconfigured config). ADR-0012. Tests: block relocation with a full ECO
engagement at 0x500, neutral API, rule-40 C/Python parity.

Clocking: tools/clock_tree.py evaluates 28 complete clock trees x 4 bus
cases from ST register widths and HAL ranges; the v0.2 "40 MHz required"
claim is withdrawn and the crystal is unselected until the bus is known.

Schematic: INA228 pins renumbered (KiCad-library cross-check, secondary);
DRV8353S stays an explicit placeholder; crystal unselected; PWR_FLAGs added
after a new pin-type check (not an ERC) found 6 undriven-rail errors.
Real KiCad ERC not run (KiCad 7 has no CLI ERC; tools/run_kicad_erc.sh).

Telematics: combined architecture with the STM32U575 / CAN 2.0B / LTE-MQTT
proposal (supervisor and CSIA placement, torque-request and driver-
authorization paths, pit/cloud outside the control chain), interface
difference table, generated DBC, logging-capacity and auxiliary-power
budget. Validation language separates command ceilings, envelope ramp,
phase current and battery current. CSIA: component attribution and a
next-evaluation plan; frozen results unchanged, nothing re-run.

Verified on the host: ctest 6/6 (4,006 checks), pytest 199 passed,
ARM core build 0 warnings, generators current, KiCad connectivity 0
problems. Nothing on hardware.

Co-Authored-By: Claude Opus 5.5 <noreply@anthropic.com>
Claude-Ses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
Changed lines of the file:
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@@
     (pin "3")
   )
-  (symbol (lib_id "Device:Q_NMOS_GDS") (at 462.28000000000003 66.04 0) (unit 1)
+  (symbol (lib_id "Device:Q_NMOS_GDS") (at 462.28 66.04 0) (unit 1)
     (in_bom yes) (on_board yes)
-    (property "Reference" "Q304" (id 0) (at 462.28000000000003 60.96000000000001 0)
+    (property "Reference" "Q304" (id 0) (at 462.28 60.96000000000001 0)
       (effects (font (size 1.27 1.27)))
     )
-    (property "Value" "UNRESOLVED N-MOSFET LS-B" (id 1) (at 462.28000000000003 71.12 0)
+    (property "Value" "UNRESOLVED N-MOSFET LS-B" (id 1) (at 462.28 71.12 0)
       (effects (font (size 1.27 1.27)))
     )
-    (property "Footprint" "" (id 2) (at 462.28000000000003 66.04 0)
+    (property "Footprint" "" (id 2) (at 462.28 66.04 0)
       (effects (font (size 1.27 1.27)) hide)
     )
-    (property "Datasheet" "" (id 3) (at 462.28000000000003 66.04 0)
+    (property "Datasheet" "" (id 3) (at 462.28 66.04 0)
       (effects (font (size 1.27 1.27)) hide)
     )
-    (property "Status" "UNRESOLVED" (id 4) (at 462.28000000000003 66.04 0)
+    (property "Status" "UNRESOLVED" (id 4) (at 462.28 66.04 0)
       (effects (font (size 1.27 1.27)) hide)
     )
-    (property "Rating_basis" "as HS" (id 5) (at 462.28000000000003 66.04 0)
+    (property "Rating_basis" "as HS" (id 5) (at 462.28 66.04 0)
       (effects (font (size 1.27 1.27)) hide)
     )

Commit message: hardware: footprint disposition for every BOM line, 82 assigned and checked
hardware/footprints/assignments.yaml gives each of the 122 BOM lines one
disposition. 68 lines are generic parts defined by value and package and
get a verified footprint (37 without the test points); 14 are specific
devices whose footprint is assigned from the KiCad 8.0.9 library but whose
manufacturer package drawing is unread (the LM5164 land pattern is drawn
from ST's L5973D HSOP-8 and the LQFP-100 from NXP's SOT407-1, so both must
be compared); 40 have none and say why: 28 rating-dependent, 4 waiting for a
data sheet value or pin voltage, 6 connectors, 2 placeholder pinouts.
Before this change no line had a footprint.

tools/check_footprints.py fetches the 25 footprint files used, pins them by
SHA-256, and checks per reference: numbered pads equal the symbol's pin
numbers, courtyard and fabrication outline present (copper-only jumpers and
net ties excepted), SMD or through-hole, package in the name for chip
parts, the symbol's footprint filters (as KiCad's ERC does), and pin 1 = K
on diode and LED symbols. Mutation tests cover a wrong pad count, a filter
miss, a package mismatch, a missing reference and a verified line without
a footprint. Small passives on battery-voltage nets (R104, R201, R202,
R1201) were kept rating-dependent rather than given an 0603.

The generator writes the footprints into the schematic and a footprint
column into the draft BOM; hw_consistency adds BM3 (netlist footprint
equals the BOM line's); price_bom takes footprint and package from the
assignment. Pricing rules fixed where lines matched the wrong rule: LEDs
were priced as buck inductors, crystal load capacitors as 100 V MLCCs, the
UART bench header as a harness connector, the reset switch and the Zener
under one generic rule; 22 uF and 4.7 uF now 1206 and 0805 for DC bias. One
board's parts move from $89-$239 to $88-$233. A project fp-lib-table and
the CI and ERC steps fetch the pinned footprints so the ERC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
Parts:
- R301, R302, R304, R305, R307, R308: footprint (none) -> Resistor_SMD:R_0603_1608Metric
Changed lines of the file:
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@@
       (effects (font (size 1.27 1.27)))
     )
-    (property "Footprint" "" (id 2) (at 205.74 66.04 0)
+    (property "Footprint" "Resistor_SMD:R_0603_1608Metric" (id 2) (at 205.74 66.04 0)
       (effects (font (size 1.27 1.27)) hide)
     )
@@
       (effects (font (size 1.27 1.27)))
     )
-    (property "Footprint" "" (id 2) (at 264.16 66.04 0)
+    (property "Footprint" "Resistor_SMD:R_0603_1608Metric" (id 2) (at 264.16 66.04 0)
       (effects (font (size 1.27 1.27)) hide)
     )
@@
       (effects (font (size 1.27 1.27)))
     )
-    (property "Footprint" "" (id 2) (at 71.12 101.6 0)
+    (property "Footprint" "Resistor_SMD:R_0603_1608Metric" (id 2) (at 71.12 101.6 0)
       (effects (font (size 1.27 1.27)) hide)
     )
@@
       (effects (font (size 1.27 1.27)))
     )
-    (property "Footprint" "" (id 2) (at 129.54 101.6 0)
+    (property "Footprint" "Resistor_SMD:R_0603_1608Metric" (id 2) (at 129.54 101.6 0)
       (effects (font (size 1.27 1.27)) hide)
     )
@@
       (effects (font (size 1.27 1.27)))
     )
-    (property "Footprint" "" (id 2) (at 388.62 101.6 0)
+    (property "Footprint" "Resistor_SMD:R_0603_1608Metric" (id 2) (at 388.62 101.6 0)
       (effects (font (size 1.27 1.27)) hide)
     )
@@
       (effects (font (size 1.27 1.27)))
     )
-    (property "Footprint" "" (id 2) (at 449.58 101.6 0)
-      (effects (font (size 1.27 1.27)) hide)
-    )
+    (property "Footprint" "Resistor_SMD:R_0603_1608Metric" (id 2) (at 449.58 101.6 0)
+      (effects (font (size 1.27 1.27)) hide)
+    )
