File: hardware/kicad/04_gate_drive.kicad_sch (KiCad schematic)
At the start: 17 parts, among them U401 DRV8353S (candidate), U402 74LVC1G08

Commit message: sem-motor-controller v0.3: vehicle-interface provenance, transport-neutral core, clock trees, schematic checks
Provenance: the Cornell repositories are reference projects. Every place
that treated CHUDS / CAN FD / its VCU / 40 MHz as our vehicle is relabelled
or corrected (docs/PROVENANCE_AUDIT.md); the v0.2 checkpoint is preserved
with an errata banner.

Firmware: the core is transport-neutral (mc_core_on_msg_rx /
mc_core_msg_tx_poll / mc_core_on_link_state). CAN is one binding
(src/transport/mc_can_binding.c) whose 64-identifier block base is the new
calibration parameter supervision.can_id_base (id 164, rule 40, null in the
unconfigured config). ADR-0012. Tests: block relocation with a full ECO
engagement at 0x500, neutral API, rule-40 C/Python parity.

Clocking: tools/clock_tree.py evaluates 28 complete clock trees x 4 bus
cases from ST register widths and HAL ranges; the v0.2 "40 MHz required"
claim is withdrawn and the crystal is unselected until the bus is known.

Schematic: INA228 pins renumbered (KiCad-library cross-check, secondary);
DRV8353S stays an explicit placeholder; crystal unselected; PWR_FLAGs added
after a new pin-type check (not an ERC) found 6 undriven-rail errors.
Real KiCad ERC not run (KiCad 7 has no CLI ERC; tools/run_kicad_erc.sh).

Telematics: combined architecture with the STM32U575 / CAN 2.0B / LTE-MQTT
proposal (supervisor and CSIA placement, torque-request and driver-
authorization paths, pit/cloud outside the control chain), interface
difference table, generated DBC, logging-capacity and auxiliary-power
budget. Validation language separates command ceilings, envelope ramp,
phase current and battery current. CSIA: component attribution and a
next-evaluation plan; frozen results unchanged, nothing re-run.

Verified on the host: ctest 6/6 (4,006 checks), pytest 199 passed,
ARM core build 0 warnings, generators current, KiCad connectivity 0
problems. Nothing on hardware.

Co-Authored-By: Claude Opus 5.5 <noreply@anthropic.com>
Claude-Ses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
Changed lines of the file:
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@@
     (pin "2")
   )
-  (symbol (lib_id "Device:R") (at 398.78000000000003 144.78 0) (unit 1)
+  (symbol (lib_id "Device:R") (at 398.78 144.78 0) (unit 1)
     (in_bom no) (on_board yes) (dnp yes)
-    (property "Reference" "R406" (id 0) (at 398.78000000000003 139.7 0)
+    (property "Reference" "R406" (id 0) (at 398.78 139.7 0)
       (effects (font (size 1.27 1.27)))
     )
-    (property "Value" "100k" (id 1) (at 398.78000000000003 149.86 0)
+    (property "Value" "100k" (id 1) (at 398.78 149.86 0)
       (effects (font (size 1.27 1.27)))
     )
-    (property "Footprint" "" (id 2) (at 398.78000000000003 144.78 0)
+    (property "Footprint" "" (id 2) (at 398.78 144.78 0)
       (effects (font (size 1.27 1.27)) hide)
     )
-    (property "Datasheet" "" (id 3) (at 398.78000000000003 144.78 0)
+    (property "Datasheet" "" (id 3) (at 398.78 144.78 0)
       (effects (font (size 1.27 1.27)) hide)
     )
-    (property "Status" "DNP if internal pull-downs verified" (id 4) (at 398.78000000000003 144.78 0)
+    (property "Status" "DNP if internal pull-downs verified" (id 4) (at 398.78 144.78 0)
       (effects (font (size 1.27 1.27)) hide)
     )

Commit message: hardware: design review, OV comparator hysteresis fix, test points, KiCad 8.0.9 libraries
hardware/review/DESIGN_REVIEW.md reviews the draft item by item (gate
driver, MOSFETs, DC link, current sensing, hardware overcurrent,
over/undervoltage, temperature, precharge, enable defaults and
watchdog, emergency interface, DC-DC, CAN, clock, debug and test
points) with an evidence level per statement, and records what each
open item needs.

Schematic changes that need no vehicle data:
- the over-voltage comparator's hysteresis resistor went straight onto
  the TL431 node, whose low impedance made the hysteresis undefined;
  the + input is now fed through 10 k and 390 k from the output sets
  -2.5 % / +0.8 % around the reference;
- the TL431 bias is 470 ohm (1.7 mA) instead of 1 k (0.8 mA), above
  its minimum cathode current (recalled; to confirm in the datasheet);
- the six pull-downs on the gate-signal inputs are fitted until the
  driver's own pull-downs are verified;
- 21 test points for the signals the acceptance procedures probe.
Connectivity: 136 intended nets, 0 problems; pin types 0 findings;
consistency 14 PASS, 4 OPEN.

The nine KiCad 8.0.9 ERC warnings were each compared with the library:
PWR_FLAG pin name, TL431 drawing, STM32G474 symbol geometry and the
NUP2105L datasheet URL changed between the 7.0.11 library the
schematic embedded and 8.0.9; no pin number, connected name, type or
net changed. The schematic is now generated from a pinned, SHA-256
checked copy of the 8.0.9 libraries (tools/fetch_kicad_symbols.py),
which the ERC also reads; KiCad 8's (hide yes) spelling is converted
for kiutils so no field becomes visible. Both CI jobs use KiCad 8.

Firmware: the brake switch type is a calibration value; a separate
bench image (semmc_stm32g474_pwmtest) switches the gate signals at
fixed duties with DRV_ENABLE held low for acceptance stage 4; g_bench
also reports the input states.

Co-Authored-By: Claude Opus 5.5 <noreply@anthropic.com>
Claude-Session: https:/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
Parts:
- added TP401: PWM_A_HI, symbol Connector:TestPoint
- added TP402: PWM_A_LO, symbol Connector:TestPoint
- added TP403: PWM_B_HI, symbol Connector:TestPoint
- added TP404: PWM_B_LO, symbol Connector:TestPoint
- added TP405: PWM_C_HI, symbol Connector:TestPoint
- added TP406: PWM_C_LO, symbol Connector:TestPoint
- added TP407: MCU_DRV_EN, symbol Connector:TestPoint
- added TP408: DRV_EN_GATED, symbol Connector:TestPoint
- added TP409: VCP, symbol Connector:TestPoint
- added TP410: DVDD, symbol Connector:TestPoint
- R405, R406, R407, R408, R409, R410: Rating_basis (none) -> holds the gate-signal input low while the MCU pin is high-i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; Status DNP if internal pull-downs verified -> design value; now fitted; now in the parts list
Connections:
- net DRV_EN_GATED: now also TP408.1
- net DVDD: now also TP410.1
- net MCU_DRV_EN: now also TP407.1
- net PWM_A_HI: now also TP401.1
- net PWM_A_LO: now also TP402.1
- net PWM_B_HI: now also TP403.1
- net PWM_B_LO: now also TP404.1
- net PWM_C_HI: now also TP405.1
- net PWM_C_LO: now also TP406.1
- net VCP: now also TP409.1

Commit message: hardware: footprint disposition for every BOM line, 82 assigned and checked
hardware/footprints/assignments.yaml gives each of the 122 BOM lines one
disposition. 68 lines are generic parts defined by value and package and
get a verified footprint (37 without the test points); 14 are specific
devices whose footprint is assigned from the KiCad 8.0.9 library but whose
manufacturer package drawing is unread (the LM5164 land pattern is drawn
from ST's L5973D HSOP-8 and the LQFP-100 from NXP's SOT407-1, so both must
be compared); 40 have none and say why: 28 rating-dependent, 4 waiting for a
data sheet value or pin voltage, 6 connectors, 2 placeholder pinouts.
Before this change no line had a footprint.

tools/check_footprints.py fetches the 25 footprint files used, pins them by
SHA-256, and checks per reference: numbered pads equal the symbol's pin
numbers, courtyard and fabrication outline present (copper-only jumpers and
net ties excepted), SMD or through-hole, package in the name for chip
parts, the symbol's footprint filters (as KiCad's ERC does), and pin 1 = K
on diode and LED symbols. Mutation tests cover a wrong pad count, a filter
miss, a package mismatch, a missing reference and a verified line without
a footprint. Small passives on battery-voltage nets (R104, R201, R202,
R1201) were kept rating-dependent rather than given an 0603.

The generator writes the footprints into the schematic and a footprint
column into the draft BOM; hw_consistency adds BM3 (netlist footprint
equals the BOM line's); price_bom takes footprint and package from the
assignment. Pricing rules fixed where lines matched the wrong rule: LEDs
were priced as buck inductors, crystal load capacitors as 100 V MLCCs, the
UART bench header as a harness connector, the reset switch and the Zener
under one generic rule; 22 uF and 4.7 uF now 1206 and 0805 for DC bias. One
board's parts move from $89-$239 to $88-$233. A project fp-lib-table and
the CI and ERC steps fetch the pinned footprints so the ERC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
Parts:
- R401, R402, R403, R404, R405, R406, R407, R408, R409, R410: footprint (none) -> Resistor_SMD:R_0603_1608Metric
- TP401, TP402, TP403, TP404, TP405, TP406, TP407, TP408, TP409, TP410: footprint (none) -> TestPoint:TestPoint_Pad_D1.5mm
- U402: footprint (none) -> Package_TO_SOT_SMD:SOT-23-5
Changed lines of the file:
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@@
       (effects (font (size 1.27 1.27)))
     )
-    (property "Footprint" "" (id 2) (at 459.74 66.04 0)
+    (property "Footprint" "Resistor_SMD:R_0603_1608Metric" (id 2) (at 459.74 66.04 0)
       (effects (font (size 1.27 1.27)) hide)
     )
@@
       (effects (font (size 1.27 1.27)))
     )
-    (property "Footprint" "" (id 2) (at 86.36 149.86 0)
+    (property "Footprint" "Package_TO_SOT_SMD:SOT-23-5" (id 2) (at 86.36 149.86 0)
       (effects (font (size 1.27 1.27)) hide)
     )
@@
       (effects (font (size 1.27 1.27)))
     )
-    (property "Footprint" "" (id 2) (at 157.48 144.78 0)
+    (property "Footprint" "Resistor_SMD:R_0603_1608Metric" (id 2) (at 157.48 144.78 0)
       (effects (font (size 1.27 1.27)) hide)
     )
@@
       (effects (font (size 1.27 1.27)))
     )
-    (property "Footprint" "" (id 2) (at 218.44 144.78 0)
+    (property "Footprint" "Resistor_SMD:R_0603_1608Metric" (id 2) (at 218.44 144.78 0)
       (effects (font (size 1.27 1.27)) hide)
     )
@@
       (effects (font (size 1.27 1.27)))
     )
-    (property "Footprint" "" (id 2) (at 276.86 144.78 0)
+    (property "Footprint" "Resistor_SMD:R_0603_1608Metric" (id 2) (at 276.86 144.78 0)
       (effects (font (size 1.27 1.27)) hide)
     )
@@
       (effects (font (size 1.27 1.27)))
     )
-    (property "Footprint" "" (id 2) (at 337.82 144.78 0)
+    (property "Footprint" "Resistor_SMD:R_0603_1608Metric" (id 2) (at 337.82 144.78 0)
       (effects (font (size 1.27 1.27)) hide)
     )
@@
       (effects (font (size 1.27 1.27)))
     )
-    (property "Footprint" "" (id 2) (at 398.78 144.78 0)
+    (property "Footprint" "Resistor_SMD:R_0603_1608Metric" (id 2) (at 398.78 144.78 0)
       (effects (font (size 1.27 1.27)) hide)
     )
@@
       (effects (font (size 1.27 1.27)))
     )
-    (property "Footprint" "" (id 2) (at 457.2 144.78 0)
+    (property "Footprint" "Resistor_SMD:R_0603_1608Metric" (id 2) (at 457.2 144.78 0)
       (effects (font (size 1.27 1.27)) hide)
     )
@@
       (effects (font (size 1.27 1.27)))
     )
-    (property "Footprint" "" (id 2) (at 71.12 190.5 0)
+    (property "Footprint" "Resistor_SMD:R_0603_1608Metric" (id 2) (at 71.12 190.5 0)
       (effects (font (size 1.27 1.27)) hide)
     )
@@
       (effects (font (size 1.27 1.27)))
     )
-    (property "Footprint" "" (id 2) (at 129.54 190.5 0)
+    (property "Footprint" "Resistor_SMD:R_0603_1608Metric" (id 2) (at 129.54 190.5 0)
       (effects (font (size 1.27 1.27)) hide)
     )
@@
       (effects (font (size 1.27 1.27)))
     )
-    (property "Footprint" "" (id 2) (at 190.5 190.5 0)
+    (property "Footprint" "Resistor_SMD:R_0603_1608Metric" (id 2) (at 190.5 190.5 0)
       (effects (font (size 1.27 1.27)) hide)
     )
@@
       (effects (font (size 1.27 1.27)))
     )
-    (property "Footprint" "" (id 2) (at 248.92 185.42 0)
+    (property "Footprint" "TestPoint:TestPoint_Pad_D1.5mm" (id 2) (at 248.92 185.42 0)
       (effects (font (size 1.27 1.27)) hide)
     )
@@
       (effects (font (size 1.27 1.27)))
     )
-    (property "Footprint" "" (id 2) (at 309.88 185.42 0)
+    (property "Footprint" "TestPoint:TestPoint_Pad_D1.5mm" (id 2) (at 309.88 185.42 0)
       (effects (font (size 1.27 1.27)) hide)
     )
@@
       (effects (font (size 1.27 1.27)))
     )
-    (property "Footprint" "" (id 2) (at 370.84 185.42 0)
+    (property "Footprint" "TestPoint:TestPoint_Pad_D1.5mm" (id 2) (at 370.84 185.42 0)
       (effects (font (size 1.27 1.27)) hide)
     )
@@
       (effects (font (size 1.27 1.27)))
     )
-    (property "Footprint" "" (id 2) (at 429.26 185.42 0)
+    (property "Footprint" "TestPoint:TestPoint_Pad_D1.5mm" (id 2) (at 429.26 185.42 0)
       (effects (font (size 1.27 1.27)) hide)
     )
@@
       (effects (font (size 1.27 1.27)))
     )
-    (property "Footprint" "" (id 2) (at 490.22 185.42 0)
+    (property "Footprint" "TestPoint:TestPoint_Pad_D1.5mm" (id 2) (at 490.22 185.42 0)
       (effects (font (size 1.27 1.27)) hide)
     )
@@
       (effects (font (size 1.27 1.27)))
     )
-    (property "Footprint" "" (id 2) (at 71.12 218.44 0)
+    (property "Footprint" "TestPoint:TestPoint_Pad_D1.5mm" (id 2) (at 71.12 218.44 0)
       (effects (font (size 1.27 1.27)) hide)
     )
@@
       (effects (font (size 1.27 1.27)))
     )
-    (property "Footprint" "" (id 2) (at 129.54 218.44 0)
+    (property "Footprint" "TestPoint:TestPoint_Pad_D1.5mm" (id 2) (at 129.54 218.44 0)
       (effects (font (size 1.27 1.27)) hide)
     )
@@
       (effects (font (size 1.27 1.27)))
     )
-    (property "Footprint" "" (id 2) (at 190.5 218.44 0)
+    (property "Footprint" "TestPoint:TestPoint_Pad_D1.5mm" (id 2) (at 190.5 218.44 0)
       (effects (font (size 1.27 1.27)) hide)
     )
@@
       (effects (font (size 1.27 1.27)))
     )
-    (property "Footprint" "" (id 2) (at 248.92 218.44 0)
+    (property "Footprint" "TestPoint:TestPoint_Pad_D1.5mm" (id 2) (at 248.92 218.44 0)
       (effects (font (size 1.27 1.27)) hide)
     )
@@
       (effects (font (size 1.27 1.27)))
     )
-    (property "Footprint" "" (id 2) (at 309.88 218.44 0)
-      (effects (font (size 1.27 1.27)) hide)
-    )
+    (property "Footprint" "TestPoint:TestPoint_Pad_D1.5mm" (id 2) (at 309.88 218.44 0)
+      (effects (font (size 1.27 1.27)) hide)
+    )
