File: hardware/kicad/05_current_sense.kicad_sch (KiCad schematic)
At the start: 12 parts

Commit message: sem-motor-controller v0.3: vehicle-interface provenance, transport-neutral core, clock trees, schematic checks
Provenance: the Cornell repositories are reference projects. Every place
that treated CHUDS / CAN FD / its VCU / 40 MHz as our vehicle is relabelled
or corrected (docs/PROVENANCE_AUDIT.md); the v0.2 checkpoint is preserved
with an errata banner.

Firmware: the core is transport-neutral (mc_core_on_msg_rx /
mc_core_msg_tx_poll / mc_core_on_link_state). CAN is one binding
(src/transport/mc_can_binding.c) whose 64-identifier block base is the new
calibration parameter supervision.can_id_base (id 164, rule 40, null in the
unconfigured config). ADR-0012. Tests: block relocation with a full ECO
engagement at 0x500, neutral API, rule-40 C/Python parity.

Clocking: tools/clock_tree.py evaluates 28 complete clock trees x 4 bus
cases from ST register widths and HAL ranges; the v0.2 "40 MHz required"
claim is withdrawn and the crystal is unselected until the bus is known.

Schematic: INA228 pins renumbered (KiCad-library cross-check, secondary);
DRV8353S stays an explicit placeholder; crystal unselected; PWR_FLAGs added
after a new pin-type check (not an ERC) found 6 undriven-rail errors.
Real KiCad ERC not run (KiCad 7 has no CLI ERC; tools/run_kicad_erc.sh).

Telematics: combined architecture with the STM32U575 / CAN 2.0B / LTE-MQTT
proposal (supervisor and CSIA placement, torque-request and driver-
authorization paths, pit/cloud outside the control chain), interface
difference table, generated DBC, logging-capacity and auxiliary-power
budget. Validation language separates command ceilings, envelope ramp,
phase current and battery current. CSIA: component attribution and a
next-evaluation plan; frozen results unchanged, nothing re-run.

Verified on the host: ctest 6/6 (4,006 checks), pytest 199 passed,
ARM core build 0 warnings, generators current, KiCad connectivity 0
problems. Nothing on hardware.

Co-Authored-By: Claude Opus 5.5 <noreply@anthropic.com>
Claude-Ses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
Other:
- note added: "PROPOSED, not substantiated: phase currents to ADC1, ADC2 and ADC3 started by the same TIM1 trigger. Simultaneity still needs the trigger configuration, ADC synchronization, acquisition windows and a bench measurement (hardware/timing/timing_budget.md, bring-up stage 4)."
- note removed: "Phase currents go to ADC1, ADC2 and ADC3, which are started by the same TIM1 trigger: the samples are simultaneous (hardware/timing/MCU_TIMING_ALLOCATION.md)."
Changed lines of the file:
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@@
     (comment 2 "Pin_check UNVERIFIED = pinout not checked against a primary datasheet")
   )
-  (text "Phase currents go to ADC1, ADC2 and ADC3, which are started by the same TIM1 trigger: the samples are simultaneous (hardware/timing/MCU_TIMING_ALLOCATION.md)."
+  (text "PROPOSED, not substantiated: phase currents to ADC1, ADC2 and ADC3 started by the same TIM1 trigger. Simultaneity still needs the trigger configuration, ADC synchronization, acquisition windows and a bench measurement (hardware/timing/timing_budget.md, bring-up stage 4)."
     (at 20.0 20.0 0)
     (effects (font (size 1.8 1.8)) (justify left))
@@
     (pin "2")
   )
-  (symbol (lib_id "Connector:TestPoint") (at 248.92000000000002 60.96 0) (unit 1)
-    (in_bom yes) (on_board yes)
-    (property "Reference" "TP501" (id 0) (at 248.92000000000002 55.88 0)
-      (effects (font (size 1.27 1.27)))
-    )
-    (property "Value" "ISENSE_A" (id 1) (at 248.92000000000002 66.04 0)
-      (effects (font (size 1.27 1.27)))
-    )
-    (property "Footprint" "" (id 2) (at 248.92000000000002 60.96 0)
-      (effects (font (size 1.27 1.27)) hide)
-    )
-    (property "Datasheet" "" (id 3) (at 248.92000000000002 60.96 0)
-      (effects (font (size 1.27 1.27)) hide)
-    )
-    (property "Status" "bench test point" (id 4) (at 248.92000000000002 60.96 0)
+  (symbol (lib_id "Connector:TestPoint") (at 248.92 60.96 0) (unit 1)
+    (in_bom yes) (on_board yes)
+    (property "Reference" "TP501" (id 0) (at 248.92 55.88 0)
+      (effects (font (size 1.27 1.27)))
+    )
+    (property "Value" "ISENSE_A" (id 1) (at 248.92 66.04 0)
+      (effects (font (size 1.27 1.27)))
+    )
+    (property "Footprint" "" (id 2) (at 248.92 60.96 0)
+      (effects (font (size 1.27 1.27)) hide)
+    )
+    (property "Datasheet" "" (id 3) (at 248.92 60.96 0)
+      (effects (font (size 1.27 1.27)) hide)
+    )
+    (property "Status" "bench test point" (id 4) (at 248.92 60.96 0)
       (effects (font (size 1.27 1.27)) hide)
     )
@@
     (pin "2")
   )
-  (symbol (lib_id "Device:R") (at 370.84000000000003 66.04 0) (unit 1)
-    (in_bom yes) (on_board yes)
-    (property "Reference" "R502" (id 0) (at 370.84000000000003 60.96000000000001 0)
-      (effects (font (size 1.27 1.27)))
-    )
-    (property "Value" "100R" (id 1) (at 370.84000000000003 71.12 0)
-      (effects (font (size 1.27 1.27)))
-    )
-    (property "Footprint" "" (id 2) (at 370.84000000000003 66.04 0)
-      (effects (font (size 1.27 1.27)) hide)
-    )
-    (property "Datasheet" "" (id 3) (at 370.84000000000003 66.04 0)
-      (effects (font (size 1.27 1.27)) hide)
-    )
-    (property "Status" "design value - see timing budget" (id 4) (at 370.84000000000003 66.04 0)
-      (effects (font (size 1.27 1.27)) hide)
-    )
-    (property "Rating_basis" "with 470 pF: tau = 47 ns (settling inside the PWM sampling window)" (id 5) (at 370.84000000000003 66.04 0)
+  (symbol (lib_id "Device:R") (at 370.84 66.04 0) (unit 1)
+    (in_bom yes) (on_board yes)
+    (property "Reference" "R502" (id 0) (at 370.84 60.96000000000001 0)
+      (effects (font (size 1.27 1.27)))
+    )
+    (property "Value" "100R" (id 1) (at 370.84 71.12 0)
+      (effects (font (size 1.27 1.27)))
+    )
+    (property "Footprint" "" (id 2) (at 370.84 66.04 0)
+      (effects (font (size 1.27 1.27)) hide)
+    )
+    (property "Datasheet" "" (id 3) (at 370.84 66.04 0)
+      (effects (font (size 1.27 1.27)) hide)
+    )
+    (property "Status" "design value - see timing budget" (id 4) (at 370.84 66.04 0)
+      (effects (font (size 1.27 1.27)) hide)
+    )
+    (property "Rating_basis" "with 470 pF: tau = 47 ns (settling inside the PWM sampling window)" (id 5) (at 370.84 66.04 0)
       (effects (font (size 1.27 1.27)) hide)
     )
@@
     (pin "2")
   )
-  (symbol (lib_id "Connector:TestPoint") (at 248.92000000000002 93.98 0) (unit 1)
-    (in_bom yes) (on_board yes)
-    (property "Reference" "TP503" (id 0) (at 248.92000000000002 88.9 0)
-      (effects (font (size 1.27 1.27)))
-    )
-    (property "Value" "ISENSE_C" (id 1) (at 248.92000000000002 99.06 0)
-      (effects (font (size 1.27 1.27)))
-    )
-    (property "Footprint" "" (id 2) (at 248.92000000000002 93.98 0)
-      (effects (font (size 1.27 1.27)) hide)
-    )
-    (property "Datasheet" "" (id 3) (at 248.92000000000002 93.98 0)
-      (effects (font (size 1.27 1.27)) hide)
-    )
-    (property "Status" "bench test point" (id 4) (at 248.92000000000002 93.98 0)
-      (effects (font (size 1.27 1.27)) hide)
-    )
+  (symbol (lib_id "Connector:TestPoint") (at 248.92 93.98 0) (unit 1)
+    (in_bom yes) (on_board yes)
+    (property "Reference" "TP503" (id 0) (at 248.92 88.9 0)
+      (effects (font (size 1.27 1.27)))
+    )
+    (property "Value" "ISENSE_C" (id 1) (at 248.92 99.06 0)
+      (effects (font (size 1.27 1.27)))
+    )
+    (property "Footprint" "" (id 2) (at 248.92 93.98 0)
+      (effects (font (size 1.27 1.27)) hide)
+    )
+    (property "Datasheet" "" (id 3) (at 248.92 93.98 0)
+      (effects (font (size 1.27 1.27)) hide)
+    )
+    (property "Status" "bench test point" (id 4) (at 248.92 93.98 0)
+      (effects (font (size 1.27 1.27)) hide)
+    )

Commit message: hardware: footprint disposition for every BOM line, 82 assigned and checked
hardware/footprints/assignments.yaml gives each of the 122 BOM lines one
disposition. 68 lines are generic parts defined by value and package and
get a verified footprint (37 without the test points); 14 are specific
devices whose footprint is assigned from the KiCad 8.0.9 library but whose
manufacturer package drawing is unread (the LM5164 land pattern is drawn
from ST's L5973D HSOP-8 and the LQFP-100 from NXP's SOT407-1, so both must
be compared); 40 have none and say why: 28 rating-dependent, 4 waiting for a
data sheet value or pin voltage, 6 connectors, 2 placeholder pinouts.
Before this change no line had a footprint.

tools/check_footprints.py fetches the 25 footprint files used, pins them by
SHA-256, and checks per reference: numbered pads equal the symbol's pin
numbers, courtyard and fabrication outline present (copper-only jumpers and
net ties excepted), SMD or through-hole, package in the name for chip
parts, the symbol's footprint filters (as KiCad's ERC does), and pin 1 = K
on diode and LED symbols. Mutation tests cover a wrong pad count, a filter
miss, a package mismatch, a missing reference and a verified line without
a footprint. Small passives on battery-voltage nets (R104, R201, R202,
R1201) were kept rating-dependent rather than given an 0603.

The generator writes the footprints into the schematic and a footprint
column into the draft BOM; hw_consistency adds BM3 (netlist footprint
equals the BOM line's); price_bom takes footprint and package from the
assignment. Pricing rules fixed where lines matched the wrong rule: LEDs
were priced as buck inductors, crystal load capacitors as 100 V MLCCs, the
UART bench header as a harness connector, the reset switch and the Zener
under one generic rule; 22 uF and 4.7 uF now 1206 and 0805 for DC bias. One
board's parts move from $89-$239 to $88-$233. A project fp-lib-table and
the CI and ERC steps fetch the pinned footprints so the ERC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
Parts:
- C501, C502, C503, C504, C505, C506: footprint (none) -> Capacitor_SMD:C_0603_1608Metric
- R501, R502, R503: footprint (none) -> Resistor_SMD:R_0603_1608Metric
- TP501, TP502, TP503: footprint (none) -> TestPoint:TestPoint_Pad_D1.5mm
Changed lines of the file:
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@@
       (effects (font (size 1.27 1.27)))
     )
-    (property "Footprint" "" (id 2) (at 71.12 66.04 0)
+    (property "Footprint" "Capacitor_SMD:C_0603_1608Metric" (id 2) (at 71.12 66.04 0)
       (effects (font (size 1.27 1.27)) hide)
     )
@@
       (effects (font (size 1.27 1.27)))
     )
-    (property "Footprint" "" (id 2) (at 129.54 66.04 0)
+    (property "Footprint" "Resistor_SMD:R_0603_1608Metric" (id 2) (at 129.54 66.04 0)
       (effects (font (size 1.27 1.27)) hide)
     )
@@
       (effects (font (size 1.27 1.27)))
     )
-    (property "Footprint" "" (id 2) (at 190.5 66.04 0)
+    (property "Footprint" "Capacitor_SMD:C_0603_1608Metric" (id 2) (at 190.5 66.04 0)
       (effects (font (size 1.27 1.27)) hide)
     )
@@
       (effects (font (size 1.27 1.27)))
     )
-    (property "Footprint" "" (id 2) (at 248.92 60.96 0)
+    (property "Footprint" "TestPoint:TestPoint_Pad_D1.5mm" (id 2) (at 248.92 60.96 0)
       (effects (font (size 1.27 1.27)) hide)
     )
@@
       (effects (font (size 1.27 1.27)))
     )
-    (property "Footprint" "" (id 2) (at 309.88 66.04 0)
+    (property "Footprint" "Capacitor_SMD:C_0603_1608Metric" (id 2) (at 309.88 66.04 0)
       (effects (font (size 1.27 1.27)) hide)
     )
@@
       (effects (font (size 1.27 1.27)))
     )
-    (property "Footprint" "" (id 2) (at 370.84 66.04 0)
+    (property "Footprint" "Resistor_SMD:R_0603_1608Metric" (id 2) (at 370.84 66.04 0)
       (effects (font (size 1.27 1.27)) hide)
     )
@@
       (effects (font (size 1.27 1.27)))
     )
-    (property "Footprint" "" (id 2) (at 429.26 66.04 0)
+    (property "Footprint" "Capacitor_SMD:C_0603_1608Metric" (id 2) (at 429.26 66.04 0)
       (effects (font (size 1.27 1.27)) hide)
     )
@@
       (effects (font (size 1.27 1.27)))
     )
-    (property "Footprint" "" (id 2) (at 490.22 60.96 0)
+    (property "Footprint" "TestPoint:TestPoint_Pad_D1.5mm" (id 2) (at 490.22 60.96 0)
       (effects (font (size 1.27 1.27)) hide)
     )
@@
       (effects (font (size 1.27 1.27)))
     )
-    (property "Footprint" "" (id 2) (at 71.12 99.06 0)
+    (property "Footprint" "Capacitor_SMD:C_0603_1608Metric" (id 2) (at 71.12 99.06 0)
       (effects (font (size 1.27 1.27)) hide)
     )
@@
       (effects (font (size 1.27 1.27)))
     )
-    (property "Footprint" "" (id 2) (at 129.54 99.06 0)
+    (property "Footprint" "Resistor_SMD:R_0603_1608Metric" (id 2) (at 129.54 99.06 0)
       (effects (font (size 1.27 1.27)) hide)
     )
@@
       (effects (font (size 1.27 1.27)))
     )
-    (property "Footprint" "" (id 2) (at 190.5 99.06 0)
+    (property "Footprint" "Capacitor_SMD:C_0603_1608Metric" (id 2) (at 190.5 99.06 0)
       (effects (font (size 1.27 1.27)) hide)
     )
@@
       (effects (font (size 1.27 1.27)))
     )
-    (property "Footprint" "" (id 2) (at 248.92 93.98 0)
-      (effects (font (size 1.27 1.27)) hide)
-    )
+    (property "Footprint" "TestPoint:TestPoint_Pad_D1.5mm" (id 2) (at 248.92 93.98 0)
+      (effects (font (size 1.27 1.27)) hide)
+    )
