File: hardware/kicad/08_mcu_debug.kicad_sch (KiCad schematic)
At the start: 30 parts, among them J801 SWD, J802 UART (bench), SW801 RESET, U801 STM32G474VET6, U802 MAX6369 (candidate), Y801 HSE UNSELECTED

Commit message: hardware: design review, OV comparator hysteresis fix, test points, KiCad 8.0.9 libraries
hardware/review/DESIGN_REVIEW.md reviews the draft item by item (gate
driver, MOSFETs, DC link, current sensing, hardware overcurrent,
over/undervoltage, temperature, precharge, enable defaults and
watchdog, emergency interface, DC-DC, CAN, clock, debug and test
points) with an evidence level per statement, and records what each
open item needs.

Schematic changes that need no vehicle data:
- the over-voltage comparator's hysteresis resistor went straight onto
  the TL431 node, whose low impedance made the hysteresis undefined;
  the + input is now fed through 10 k and 390 k from the output sets
  -2.5 % / +0.8 % around the reference;
- the TL431 bias is 470 ohm (1.7 mA) instead of 1 k (0.8 mA), above
  its minimum cathode current (recalled; to confirm in the datasheet);
- the six pull-downs on the gate-signal inputs are fitted until the
  driver's own pull-downs are verified;
- 21 test points for the signals the acceptance procedures probe.
Connectivity: 136 intended nets, 0 problems; pin types 0 findings;
consistency 14 PASS, 4 OPEN.

The nine KiCad 8.0.9 ERC warnings were each compared with the library:
PWR_FLAG pin name, TL431 drawing, STM32G474 symbol geometry and the
NUP2105L datasheet URL changed between the 7.0.11 library the
schematic embedded and 8.0.9; no pin number, connected name, type or
net changed. The schematic is now generated from a pinned, SHA-256
checked copy of the 8.0.9 libraries (tools/fetch_kicad_symbols.py),
which the ERC also reads; KiCad 8's (hide yes) spelling is converted
for kiutils so no field becomes visible. Both CI jobs use KiCad 8.

Firmware: the brake switch type is a calibration value; a separate
bench image (semmc_stm32g474_pwmtest) switches the gate signals at
fixed duties with DRV_ENABLE held low for acceptance stage 4; g_bench
also reports the input states.

Co-Authored-By: Claude Opus 5.5 <noreply@anthropic.com>
Claude-Session: https:/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
Parts:
- added TP804: WDG_WDI, symbol Connector:TestPoint
- added TP805: WDG_RST_N, symbol Connector:TestPoint
Connections:
- net WDG_RST_N: now also TP805.1
- net WDG_WDI: now also TP804.1
Other:
- moved on the sheet: C801, C802, C803, C804, C805, C806, C807, C808, C809, C810, C811, C812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

Commit message: hardware: footprint disposition for every BOM line, 82 assigned and checked
hardware/footprints/assignments.yaml gives each of the 122 BOM lines one
disposition. 68 lines are generic parts defined by value and package and
get a verified footprint (37 without the test points); 14 are specific
devices whose footprint is assigned from the KiCad 8.0.9 library but whose
manufacturer package drawing is unread (the LM5164 land pattern is drawn
from ST's L5973D HSOP-8 and the LQFP-100 from NXP's SOT407-1, so both must
be compared); 40 have none and say why: 28 rating-dependent, 4 waiting for a
data sheet value or pin voltage, 6 connectors, 2 placeholder pinouts.
Before this change no line had a footprint.

tools/check_footprints.py fetches the 25 footprint files used, pins them by
SHA-256, and checks per reference: numbered pads equal the symbol's pin
numbers, courtyard and fabrication outline present (copper-only jumpers and
net ties excepted), SMD or through-hole, package in the name for chip
parts, the symbol's footprint filters (as KiCad's ERC does), and pin 1 = K
on diode and LED symbols. Mutation tests cover a wrong pad count, a filter
miss, a package mismatch, a missing reference and a verified line without
a footprint. Small passives on battery-voltage nets (R104, R201, R202,
R1201) were kept rating-dependent rather than given an 0603.

The generator writes the footprints into the schematic and a footprint
column into the draft BOM; hw_consistency adds BM3 (netlist footprint
equals the BOM line's); price_bom takes footprint and package from the
assignment. Pricing rules fixed where lines matched the wrong rule: LEDs
were priced as buck inductors, crystal load capacitors as 100 V MLCCs, the
UART bench header as a harness connector, the reset switch and the Zener
under one generic rule; 22 uF and 4.7 uF now 1206 and 0805 for DC bias. One
board's parts move from $89-$239 to $88-$233. A project fp-lib-table and
the CI and ERC steps fetch the pinned footprints so the ERC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
Parts:
- C801, C802, C803, C804, C805, C807, C808, C809, C810, C811, C812: footprint (none) -> Capacitor_SMD:C_0603_1608Metric
- C806: footprint (none) -> Capacitor_SMD:C_0805_2012Metric
- D801, D802: footprint (none) -> LED_SMD:LED_0603_1608Metric
- D803: footprint (none) -> Diode_SMD:D_SOD-323
- FB801: footprint (none) -> Inductor_SMD:L_0603_1608Metric
- J801: footprint (none) -> Connector_PinHeader_1.27mm:PinHeader_2x05_P1.27mm_Vertical_SMD
- J802: footprint (none) -> Connector_PinHeader_2.54mm:PinHeader_1x03_P2.54mm_Vertical
- R801, R802, R803, R804, R805: footprint (none) -> Resistor_SMD:R_0603_1608Metric
- SW801: footprint (none) -> Button_Switch_SMD:SW_SPST_PTS645
- TP801, TP802, TP803, TP804, TP805: footprint (none) -> TestPoint:TestPoint_Pad_D1.5mm
- U801: footprint (none) -> Package_QFP:LQFP-100_14x14mm_P0.5mm
- U802: footprint (none) -> Package_TO_SOT_SMD:SOT-23-8
- Y801: footprint (none) -> Crystal:Crystal_SMD_3225-4Pin_3.2x2.5mm
Changed lines of the file:
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@@
       (effects (font (size 1.27 1.27)))
     )
-    (property "Footprint" "" (id 2) (at 93.98 134.62 0)
+    (property "Footprint" "Package_QFP:LQFP-100_14x14mm_P0.5mm" (id 2) (at 93.98 134.62 0)
       (effects (font (size 1.27 1.27)) hide)
     )
@@
       (effects (font (size 1.27 1.27)))
     )
-    (property "Footprint" "" (id 2) (at 175.26 66.04 0)
+    (property "Footprint" "Capacitor_SMD:C_0603_1608Metric" (id 2) (at 175.26 66.04 0)
       (effects (font (size 1.27 1.27)) hide)
     )
@@
       (effects (font (size 1.27 1.27)))
     )
-    (property "Footprint" "" (id 2) (at 236.22 66.04 0)
+    (property "Footprint" "Capacitor_SMD:C_0603_1608Metric" (id 2) (at 236.22 66.04 0)
       (effects (font (size 1.27 1.27)) hide)
     )
@@
       (effects (font (size 1.27 1.27)))
     )
-    (property "Footprint" "" (id 2) (at 294.64 66.04 0)
+    (property "Footprint" "Capacitor_SMD:C_0603_1608Metric" (id 2) (at 294.64 66.04 0)
       (effects (font (size 1.27 1.27)) hide)
     )
@@
       (effects (font (size 1.27 1.27)))
     )
-    (property "Footprint" "" (id 2) (at 355.6 66.04 0)
+    (property "Footprint" "Capacitor_SMD:C_0603_1608Metric" (id 2) (at 355.6 66.04 0)
       (effects (font (size 1.27 1.27)) hide)
     )
@@
       (effects (font (size 1.27 1.27)))
     )
-    (property "Footprint" "" (id 2) (at 416.56 66.04 0)
+    (property "Footprint" "Capacitor_SMD:C_0603_1608Metric" (id 2) (at 416.56 66.04 0)
       (effects (font (size 1.27 1.27)) hide)
     )
@@
       (effects (font (size 1.27 1.27)))
     )
-    (property "Footprint" "" (id 2) (at 474.98 66.04 0)
+    (property "Footprint" "Capacitor_SMD:C_0805_2012Metric" (id 2) (at 474.98 66.04 0)
       (effects (font (size 1.27 1.27)) hide)
     )
@@
       (effects (font (size 1.27 1.27)))
     )
-    (property "Footprint" "" (id 2) (at 535.94 63.5 0)
+    (property "Footprint" "Inductor_SMD:L_0603_1608Metric" (id 2) (at 535.94 63.5 0)
       (effects (font (size 1.27 1.27)) hide)
     )
@@
       (effects (font (size 1.27 1.27)))
     )
-    (property "Footprint" "" (id 2) (at 596.9 66.04 0)
+    (property "Footprint" "Capacitor_SMD:C_0603_1608Metric" (id 2) (at 596.9 66.04 0)
       (effects (font (size 1.27 1.27)) hide)
     )
@@
       (effects (font (size 1.27 1.27)))
     )
-    (property "Footprint" "" (id 2) (at 655.32 66.04 0)
+    (property "Footprint" "Capacitor_SMD:C_0603_1608Metric" (id 2) (at 655.32 66.04 0)
       (effects (font (size 1.27 1.27)) hide)
     )
@@
       (effects (font (size 1.27 1.27)))
     )
-    (property "Footprint" "" (id 2) (at 716.28 66.04 0)
+    (property "Footprint" "Capacitor_SMD:C_0603_1608Metric" (id 2) (at 716.28 66.04 0)
       (effects (font (size 1.27 1.27)) hide)
     )
@@
       (effects (font (size 1.27 1.27)))
     )
-    (property "Footprint" "" (id 2) (at 71.12 236.22 0)
+    (property "Footprint" "Resistor_SMD:R_0603_1608Metric" (id 2) (at 71.12 236.22 0)
       (effects (font (size 1.27 1.27)) hide)
     )
@@
       (effects (font (size 1.27 1.27)))
     )
-    (property "Footprint" "" (id 2) (at 129.54 236.22 0)
+    (property "Footprint" "Capacitor_SMD:C_0603_1608Metric" (id 2) (at 129.54 236.22 0)
       (effects (font (size 1.27 1.27)) hide)
     )
@@
       (effects (font (size 1.27 1.27)))
     )
-    (property "Footprint" "" (id 2) (at 195.58 231.14 0)
+    (property "Footprint" "Button_Switch_SMD:SW_SPST_PTS645" (id 2) (at 195.58 231.14 0)
       (effects (font (size 1.27 1.27)) hide)
     )
@@
       (effects (font (size 1.27 1.27)))
     )
-    (property "Footprint" "" (id 2) (at 264.16 236.22 0)
+    (property "Footprint" "Crystal:Crystal_SMD_3225-4Pin_3.2x2.5mm" (id 2) (at 264.16 236.22 0)
       (effects (font (size 1.27 1.27)) hide)
     )
@@
       (effects (font (size 1.27 1.27)))
     )
-    (property "Footprint" "" (id 2) (at 327.66 236.22 0)
+    (property "Footprint" "Capacitor_SMD:C_0603_1608Metric" (id 2) (at 327.66 236.22 0)
       (effects (font (size 1.27 1.27)) hide)
     )
@@
       (effects (font (size 1.27 1.27)))
     )
-    (property "Footprint" "" (id 2) (at 388.62 236.22 0)
+    (property "Footprint" "Capacitor_SMD:C_0603_1608Metric" (id 2) (at 388.62 236.22 0)
       (effects (font (size 1.27 1.27)) hide)
     )
@@
       (effects (font (size 1.27 1.27)))
     )
-    (property "Footprint" "" (id 2) (at 457.2 246.38 0)
+    (property "Footprint" "Connector_PinHeader_1.27mm:PinHeader_2x05_P1.27mm_Vertical_SMD" (id 2) (at 457.2 246.38 0)
       (effects (font (size 1.27 1.27)) hide)
     )
@@
       (effects (font (size 1.27 1.27)))
     )
-    (property "Footprint" "" (id 2) (at 535.94 233.68 0)
+    (property "Footprint" "Connector_PinHeader_2.54mm:PinHeader_1x03_P2.54mm_Vertical" (id 2) (at 535.94 233.68 0)
       (effects (font (size 1.27 1.27)) hide)
     )
@@
       (effects (font (size 1.27 1.27)))
     )
-    (property "Footprint" "" (id 2) (at 591.82 236.22 0)
+    (property "Footprint" "Resistor_SMD:R_0603_1608Metric" (id 2) (at 591.82 236.22 0)
       (effects (font (size 1.27 1.27)) hide)
     )
@@
       (effects (font (size 1.27 1.27)))
     )
-    (property "Footprint" "" (id 2) (at 655.32 231.14 0)
+    (property "Footprint" "LED_SMD:LED_0603_1608Metric" (id 2) (at 655.32 231.14 0)
       (effects (font (size 1.27 1.27)) hide)
     )
@@
       (effects (font (size 1.27 1.27)))
     )
-    (property "Footprint" "" (id 2) (at 718.82 236.22 0)
+    (property "Footprint" "Resistor_SMD:R_0603_1608Metric" (id 2) (at 718.82 236.22 0)
       (effects (font (size 1.27 1.27)) hide)
     )
@@
       (effects (font (size 1.27 1.27)))
     )
-    (property "Footprint" "" (id 2) (at 73.66 287.02 0)
+    (property "Footprint" "LED_SMD:LED_0603_1608Metric" (id 2) (at 73.66 287.02 0)
       (effects (font (size 1.27 1.27)) hide)
     )
@@
       (effects (font (size 1.27 1.27)))
     )
-    (property "Footprint" "" (id 2) (at 147.32 299.72 0)
+    (property "Footprint" "Package_TO_SOT_SMD:SOT-23-8" (id 2) (at 147.32 299.72 0)
       (effects (font (size 1.27 1.27)) hide)
     )
@@
       (effects (font (size 1.27 1.27)))
     )
-    (property "Footprint" "" (id 2) (at 218.44 292.1 0)
+    (property "Footprint" "Resistor_SMD:R_0603_1608Metric" (id 2) (at 218.44 292.1 0)
       (effects (font (size 1.27 1.27)) hide)
     )
@@
       (effects (font (size 1.27 1.27)))
     )
-    (property "Footprint" "" (id 2) (at 276.86 292.1 0)
+    (property "Footprint" "Resistor_SMD:R_0603_1608Metric" (id 2) (at 276.86 292.1 0)
       (effects (font (size 1.27 1.27)) hide)
     )
@@
       (effects (font (size 1.27 1.27)))
     )
-    (property "Footprint" "" (id 2) (at 342.9 287.02 0)
+    (property "Footprint" "Diode_SMD:D_SOD-323" (id 2) (at 342.9 287.02 0)
       (effects (font (size 1.27 1.27)) hide)
     )
@@
       (effects (font (size 1.27 1.27)))
     )
-    (property "Footprint" "" (id 2) (at 406.4 287.02 0)
+    (property "Footprint" "TestPoint:TestPoint_Pad_D1.5mm" (id 2) (at 406.4 287.02 0)
       (effects (font (size 1.27 1.27)) hide)
     )
@@
       (effects (font (size 1.27 1.27)))
     )
-    (property "Footprint" "" (id 2) (at 464.82 287.02 0)
+    (property "Footprint" "TestPoint:TestPoint_Pad_D1.5mm" (id 2) (at 464.82 287.02 0)
       (effects (font (size 1.27 1.27)) hide)
     )
@@
       (effects (font (size 1.27 1.27)))
     )
-    (property "Footprint" "" (id 2) (at 525.78 287.02 0)
+    (property "Footprint" "TestPoint:TestPoint_Pad_D1.5mm" (id 2) (at 525.78 287.02 0)
       (effects (font (size 1.27 1.27)) hide)
     )
@@
       (effects (font (size 1.27 1.27)))
     )
-    (property "Footprint" "" (id 2) (at 586.74 287.02 0)
+    (property "Footprint" "TestPoint:TestPoint_Pad_D1.5mm" (id 2) (at 586.74 287.02 0)
       (effects (font (size 1.27 1.27)) hide)
     )
@@
       (effects (font (size 1.27 1.27)))
     )
-    (property "Footprint" "" (id 2) (at 645.16 287.02 0)
-      (effects (font (size 1.27 1.27)) hide)
-    )
+    (property "Footprint" "TestPoint:TestPoint_Pad_D1.5mm" (id 2) (at 645.16 287.02 0)
+      (effects (font (size 1.27 1.27)) hide)
+    )
